File: Battery with Active BMS.kicad_pcb (KiCad board)
At the start: 2 copper layers, 300 x 140 mm, 102 parts, among them J1 B7B-EH-A(LF)(SN), J2 B7B-EH-A(LF)(SN), J3 B7B-EH-A(LF)(SN), P1 22-28-4033, P2 61300511121, P3 61300811121, P4 TSW-106-07-L-D, Q1 NMOS, Q2 NMOS, U1 TLI4971, U11 EL817, U16 EL817, U17 EL817, U2 ARDUINO_PRO_MINI, U3 MPC3008, U4 TC4428CPA, U5 LM78M05CT/NOPB, U8 EL817

Commit message: V0.1 Upload
Parts:
- added P5: 22-28-4033, Connector_PinHeader_2.54mm:PinHeader_2x02_P2.54mm_Vertical, F.Cu at (126.1, 38.5)
- P3: footprint Connector_PinHeader_2.54mm:PinHeader_2x07_P2.54mm_Vertical -> Connector_PinHeader_2.54mm:PinHeader_2x09_P2.54mm_Vertical
- moved P1 242.8 mm to (126.0, 109.5), turned to -90 degrees
- moved R35 230.5 mm to (129.8, 95.9), turned to 180 degrees
- moved R36 228.1 mm to (129.8, 93.4), turned to 180 degrees
- moved R37 225.7 mm to (129.7, 90.9), turned to 180 degrees
- moved R38 223.5 mm to (129.9, 88.4), turned to 180 degrees
- moved U5 220.3 mm to (84.6, 26.8), turned to 0 degrees
- moved U2 214.1 mm to (118.7, 90.9), turned to 0 degrees
- moved U8 205.7 mm to (128.5, 61.6), turned to 180 degrees
- moved R24 201.4 mm to (93.4, 54.3), turned to 90 degrees
- moved R46 200.5 mm to (127.7, 56.3), turned to 180 degrees
- moved R21 199.7 mm to (90.9, 54.3), turned to 90 degrees
- moved R20 198.1 mm to (88.4, 54.3), turned to 90 degrees
- moved R19 196.5 mm to (85.8, 54.3), turned to 90 degrees
- moved U3 195.4 mm to (75.7, 50.7), turned to 90 degrees
- moved U11 195.2 mm to (128.5, 70.6), turned to 180 degrees
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Connections:
- B1 pad 1: Net-(U1-IP+) -> Batt+
- C1 pad 2: Net-(U1-GND) -> GND
- C2 pad 2: Net-(U1-GND) -> GND
- C3 pad 2: GND -> unconnected-(C3-Pad2)
- C4 pad 2: Net-(U1-GND) -> GND
- C5 pad 2: Net-(U1-GND) -> GND
- P1 pad 2: /<NO NET> -> GND
- P1 pad 3: GND -> /<NO NET>
- P2 pad 2: /RX_{ISO} -> GND
- P2 pad 3: /TX_{ISO} -> /RX_{ISO}
- P2 pad 4: /DTR_{ISO} -> GND
- P2 pad 5: /RST_{ISO} -> /TX_{ISO}
- P2 pad 7: GND -> /DTR_{ISO}
- P2 pad 9: GND -> /RST_{ISO}
- P3 pad 11: GND -> Net-(U2-D4)
- P3 pad 13: GND -> Net-(U2-D5)
- P3 pad 2: /TX_2 -> GND
- P3 pad 3: /RX_2 -> /TX_2
- P3 pad 4: Net-(U2-D4) -> GND
- P3 pad 5: Net-(U2-D5) -> /RX_2
- P3 pad 6: Net-(U2-D6) -> GND
- P3 pad 7: Net-(U2-D7) -> Net-(U2-D2)
- P3 pad 9: GND -> Net-(U2-D3)
- U1 pad 2: Net-(U1-GND) -> GND
- U1 pad 8: Net-(U1-IP+) -> Batt+
- U2 pad JP7_7: /OCD1 -> Net-(U2-D3)
- U2 pad JP7_8: /OCD2 -> Net-(U2-D2)
- U5 pad 2: GND -> unconnected-(U5-GND-Pad2)
Routing:
- net +3.3V: track 0.00 -> 267.5 mm, vias 0 -> 2
- net /CLK: track 21.6 -> 141.9 mm
- net /DOUT: track 18.0 -> 134.1 mm
- net /DIN: track 14.8 -> 127.9 mm
- net /~{CS}: track 12.1 -> 120.6 mm
- net /AOUT: track 0.00 -> 64.1 mm, vias 0 -> 2
- net /RST: track 2.82 -> 61.1 mm
- net /VREF: track 0.00 -> 57.2 mm, vias 0 -> 2
- net Net-(U2-D8): track 18.8 -> 66.2 mm, vias 0 -> 1
- net /A4: track 0.00 -> 41.6 mm
- net Net-(U2-D9): track 11.1 -> 52.5 mm, vias 0 -> 1
- net /A5: track 0.00 -> 34.9 mm
- net /A0: track 0.00 -> 34.5 mm
- net /A2: track 0.00 -> 33.2 mm
- net /A1: track 0.00 -> 33.1 mm
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- added copper zone on B.Cu, net Batt+
- added copper zone on F.Cu, net Batt+
- added copper zone on B.Cu, net GND
- added copper zone on F.Cu, net GND
- added copper zone on F.Cu, net Net-(Q1-S)
- added copper zone on F.Cu, net Net-(Q2-D)
- added copper zone on B.Cu, net Net-(U1-IP-)
- added copper zone on F.Cu, net Net-(U1-IP-)
Other:
- board size 300 x 140 mm -> 334 x 140 mm
- board text added: "SYM"
