File: Battery with Active BMS.kicad_pcb (KiCad board)
At the start: 2 copper layers, 334 x 140 mm, 103 parts, among them J1 B7B-EH-A(LF)(SN), J2 B7B-EH-A(LF)(SN), J3 B7B-EH-A(LF)(SN), P1 22-28-4033, P2 61300511121, P3 61300811121, P4 TSW-106-07-L-D, P5 22-28-4033, Q1 NMOS, Q2 NMOS, U1 TLI4971, U11 EL817, U16 EL817, U17 EL817, U2 ARDUINO_PRO_MINI, U3 MPC3008, U4 TC4428CPA, U5 LM78M05CT/NOPB, U8 EL817

Commit message: BMS V1.0
Parts:
- added H1: MountingHole_Pad, MountingHole:MountingHole_5.3mm_M5_Pad_Via, F.Cu at (93.0, 147.0)
- added H10: MountingHole, MountingHole:MountingHole_2.5mm_Pad, F.Cu at (45.5, 150.0)
- added H11: MountingHole, MountingHole:MountingHole_2.5mm_Pad, F.Cu at (80.0, 18.0)
- added H12: MountingHole, MountingHole:MountingHole_2.5mm_Pad, F.Cu at (80.0, 101.0)
- added H2: MountingHole_Pad, MountingHole:MountingHole_5.3mm_M5_Pad_Via, F.Cu at (93.0, 101.0)
- added H3: MountingHole_Pad, MountingHole:MountingHole_5.3mm_M5_Pad_Via, F.Cu at (93.0, 21.0)
- added H4: MountingHole_Pad, MountingHole:MountingHole_5.3mm_M5_Pad_Via, F.Cu at (93.0, 67.0)
- added H5: MountingHole, MountingHole:MountingHole_2.5mm_Pad, F.Cu at (106.0, 150.0)
- added H6: MountingHole, MountingHole:MountingHole_2.5mm_Pad, F.Cu at (105.9, 18.0)
- added H7: MountingHole, MountingHole:MountingHole_2.5mm_Pad, F.Cu at (347.9, 18.4)
- added H8: MountingHole, MountingHole:MountingHole_2.5mm_Pad, F.Cu at (348.0, 150.1)
- added H9: MountingHole, MountingHole:MountingHole_2.5mm_Pad, F.Cu at (18.0, 18.0)
- B1, B2, B3, B4, B5, B6: footprint TerminalBlock_Wuerth:Wuerth_REDCUBE-THR_WP-THRBU_74650195_THR -> lib:M5 Screw Terminal
- moved B4 62.1 mm to (72.0, 33.4)
- moved B1 62.1 mm to (41.9, 33.4)
- moved B5 62.1 mm to (41.9, 143.4)
- moved B2 58.1 mm to (106.1, 143.4)
- moved B3 58.1 mm to (106.1, 33.4)
- moved R2 58.0 mm to (70.3, 46.9)
- moved R38 58.0 mm to (71.9, 88.4)
- moved U11 58.0 mm to (70.5, 70.6)
- moved U8 58.0 mm to (70.5, 61.6)
- moved P2 58.0 mm to (46.8, 62.4)
- moved U1 58.0 mm to (60.9, 36.2)
- moved U16 58.0 mm to (58.9, 61.5)
- moved U17 58.0 mm to (58.9, 70.5)
- moved U2 58.0 mm to (60.7, 90.9)
- moved U4 58.0 mm to (56.9, 141.6)
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Connections:
- C3 pad 2: unconnected-(C3-Pad2) -> GND
- U5 pad 2: unconnected-(U5-GND-Pad2) -> GND
Routing:
- net Net-(BT10--): track 246.5 -> 251.5 mm
- net Net-(BT10-+): track 169.3 -> 174.2 mm
- net Net-(BT1-+): track 96.3 -> 101.2 mm
- net Net-(BT16-+): track 18.6 -> 23.5 mm
- net Net-(BT13-+): track 90.9 -> 95.8 mm
- net Net-(BT4-+): track 168.8 -> 173.7 mm
- net /A3: track 33.1 -> 35.7 mm
- net /A0: track 34.5 -> 37.0 mm
- net /A1: track 33.1 -> 35.7 mm
- net /A2: track 33.2 -> 35.6 mm
- net +3.3V: track 267.5 -> 269.8 mm
- net /A4: track 41.6 -> 42.7 mm
- net /AOUT: track 64.1 -> 63.1 mm
- net GND: track 25.7 -> 26.2 mm, vias 2 -> 48
- net Batt+: vias 0 -> 13
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- added copper zone on B.Cu, net /Copper Conn 1
- added copper zone on F.Cu, net /Copper Conn 1
- added copper zone on B.Cu, net /Copper Conn 2
- added copper zone on F.Cu, net /Copper Conn 2
Other:
- board size 334 x 140 mm -> 338 x 140 mm

Commit message: Battery Managment System V1.0
Parts:
- removed B4: 7461383, lib:M5 Screw Terminal
- removed C1, C2, C3, C4, C5: Capacitor, Capacitor_SMD:C_0805_2012Metric_Pad1.18x1.45mm_HandSolder
- removed P5: 22-28-4033, Connector_PinHeader_2.54mm:PinHeader_2x02_P2.54mm_Vertical
- removed R26, R27: Res2, Resistor_THT:R_Axial_DIN0207_L6.3mm_D2.5mm_P10.16mm_Horizontal
- removed U1: TLI4971, Package_SON:Infineon_PG-TISON-8-5
- added BT19: Battery_Cell, lib:21700, F.Cu at (235.0, 161.0)
- added BT20: Battery_Cell, lib:21700, F.Cu at (235.0, 139.0)
- added BT21: Battery_Cell, lib:21700, F.Cu at (159.0, 161.0)
- added BT22: Battery_Cell, lib:21700, F.Cu at (159.0, 139.0)
- added BT23: Battery_Cell, lib:21700, F.Cu at (159.0, 117.0)
- added BT24: Battery_Cell, lib:21700, F.Cu at (159.0, 95.0)
- added J4: Conn_01x05_Pin, Connector_PinSocket_2.54mm:PinSocket_1x05_P2.54mm_Vertical, F.Cu at (45.9, 18.5)
- added J5: Conn_01x01_Pin, Connector_PinSocket_2.54mm:PinSocket_1x01_P2.54mm_Vertical, F.Cu at (17.8, 58.2)
- added J6: Conn_01x01_Pin, Connector_PinSocket_2.54mm:PinSocket_1x01_P2.54mm_Vertical, F.Cu at (72.5, 78.2)
- added J7: Conn_01x01_Pin, Connector_PinSocket_2.54mm:PinSocket_1x01_P2.54mm_Vertical, F.Cu at (56.0, 22.0)
- added J8: Conn_01x05_Pin, Connector_PinSocket_2.54mm:PinSocket_1x05_P2.54mm_Vertical, F.Cu at (46.0, 26.4)
- added J9: Conn_01x01_Pin, Connector_PinSocket_2.54mm:PinSocket_1x01_P2.54mm_Vertical, F.Cu at (56.1, 30.5)
- R1, R2: value Res2 -> 4.7k
- R35, R36, R37, R38, R39, R40: moved to B.Cu
- moved B1 236.7 mm to (257.2, 131.8)
- moved BT16 153.3 mm to (311.0, 161.0)
- moved BT12 132.4 mm to (311.0, 7.00), turned to -90 degrees
- moved R2 98.3 mm to (64.5, 145.0)
- moved R1 98.2 mm to (59.4, 145.0)
- moved BT11 88.4 mm to (311.0, 29.0), turned to -90 degrees
- moved BT4 79.2 mm to (159.0, 7.00)
- moved BT7 78.8 mm to (235.0, 51.0)
- moved BT8 78.8 mm to (235.0, 73.0)
- moved BT13 75.8 mm to (311.0, 139.0)
- moved BT14 75.8 mm to (311.0, 117.0)
- moved BT15 75.8 mm to (311.0, 95.0)
- moved BT17 75.8 mm to (235.0, 117.0)
- moved BT18 75.8 mm to (235.0, 95.0)
- moved BT3 44.4 mm to (159.0, 29.0)
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Connections:
- B1 pad 1: Batt+ -> Net-(BT13-+)
- B2 pad 1: Net-(BT16-+) -> Net-(BT21-+)
- BT16 pad 1: Net-(BT16-+) -> Net-(BT13-+)
- BT16 pad 2: Net-(BT13-+) -> Net-(BT10-+)
- BT17 pad 1: Net-(BT16-+) -> Net-(BT17-+)
- BT18 pad 1: Net-(BT16-+) -> Net-(BT17-+)
- BT4 pad 1: Net-(BT4-+) -> Net-(BT1-+)
- BT4 pad 2: Net-(BT1-+) -> Net-(BT1--)
- BT5 pad 1: Net-(BT4-+) -> Net-(BT10--)
- BT6 pad 1: Net-(BT4-+) -> Net-(BT10--)
- BT7 pad 2: Net-(BT4-+) -> Net-(BT1-+)
- BT8 pad 2: Net-(BT4-+) -> Net-(BT1-+)
- BT9 pad 1: Net-(BT10--) -> Net-(BT10-+)
- BT9 pad 2: Net-(BT4-+) -> Net-(BT10--)
- J1 pad 1: Net-(BT16-+) -> Net-(BT21-+)
- J1 pad 2: Net-(BT13-+) -> Net-(BT17-+)
- J1 pad 3: Net-(BT10-+) -> Net-(BT13-+)
- J1 pad 4: Net-(BT10--) -> Net-(BT10-+)
- J1 pad 5: Net-(BT4-+) -> Net-(BT10--)
- J3 pad 1: Net-(BT16-+) -> Net-(BT21-+)
- J3 pad 2: Net-(BT13-+) -> Net-(BT17-+)
- J3 pad 3: Net-(BT10-+) -> Net-(BT13-+)
- J3 pad 4: Net-(BT10--) -> Net-(BT10-+)
- J3 pad 5: Net-(BT4-+) -> Net-(BT10--)
- P1 pad 1: /A7 -> /<NO NET>
- P1 pad 3: /<NO NET> -> /A7
- P3 pad 1: /RST -> GND
- P3 pad 10: GND -> Net-(U2-D3)
- P3 pad 11: Net-(U2-D4) -> GND
- P3 pad 12: GND -> Net-(U2-D4)
- P3 pad 13: Net-(U2-D5) -> GND
- P3 pad 14: GND -> Net-(U2-D5)
- P3 pad 15: Net-(U2-D6) -> GND
- P3 pad 16: GND -> Net-(U2-D6)
- P3 pad 17: Net-(U2-D7) -> GND
- P3 pad 18: GND -> Net-(U2-D7)
- P3 pad 2: GND -> /TX_2
- P3 pad 3: /TX_2 -> GND
- P3 pad 4: GND -> /RX_2
- P3 pad 5: /RX_2 -> GND
- P3 pad 6: GND -> /RST
- P3 pad 7: Net-(U2-D2) -> GND
- P3 pad 8: GND -> Net-(U2-D2)
- P3 pad 9: Net-(U2-D3) -> GND
- P4 pad 1: /A0 -> +3.3V
- P4 pad 10: +3.3V -> /A1
- P4 pad 11: /A5 -> +3.3V
- P4 pad 12: +3.3V -> /A0
- P4 pad 2: +3.3V -> /A5
- P4 pad 3: /A1 -> +3.3V
- P4 pad 4: +3.3V -> /A4
- P4 pad 5: /A2 -> +3.3V
- P4 pad 6: +3.3V -> /A3
- P4 pad 7: /A3 -> +3.3V
- P4 pad 8: +3.3V -> /A2
- P4 pad 9: /A4 -> +3.3V
- R1 pad 1: /OCD1 -> Net-(U2-D8)
- R1 pad 2: +3.3V -> GND
- R12 pad 1: /AOUT -> Net-(J5-Pin_1)
- R16 pad 1: /VREF -> /A_{OUT}
- R2 pad 1: /OCD2 -> Net-(U2-D9)
- R2 pad 2: +3.3V -> GND
- U2 pad JP6_1: unconnected-(U2-RAW-PadJP6_1) -> Net-(J6-Pin_1)
Routing:
- net Net-(BT4-+): track 173.7 -> 0.00 mm
- net Net-(BT17-+): track 0.00 -> 95.8 mm
- net /A_{OUT}: track 0.00 -> 89.2 mm
- net Net-(BT13-+): track 95.8 -> 174.2 mm
- net Net-(BT10-+): track 174.2 -> 251.5 mm
- net Net-(BT10--): track 251.5 -> 174.6 mm
- net /AOUT: track 63.1 -> 0.00 mm, vias 2 -> 0
- net /VREF: track 57.3 -> 0.00 mm, vias 2 -> 0
- net GND: track 26.2 -> 0.00 mm, vias 48 -> 58
- net Net-(BT21-+): track 0.00 -> 23.5 mm
- net Net-(BT16-+): track 23.5 -> 0.00 mm
- net /RST: track 61.1 -> 40.2 mm
- net /OCD2: track 17.8 -> 0.00 mm
- net /OCD1: track 16.8 -> 0.00 mm
- net /~{FAULT}: track 0.00 -> 16.0 mm
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- added copper zone on B.Cu, net Net-(BT17-+)
- added copper zone on F.Cu, net Net-(BT17-+)
- added copper zone on B.Cu, net Net-(BT21-+)
- added copper zone on F.Cu, net Net-(BT21-+)
- removed copper zone on B.Cu, net Batt+
- removed copper zone on F.Cu, net Batt+
- removed copper zone on B.Cu, net Net-(BT16-+)
- removed copper zone on F.Cu, net Net-(BT16-+)
- removed copper zone on B.Cu, net Net-(BT4-+)
- removed copper zone on F.Cu, net Net-(BT4-+)
- removed copper zone on B.Cu, net Net-(U1-IP-)
- removed copper zone on F.Cu, net Net-(U1-IP-)
Other:
- board size 338 x 140 mm -> 349 x 180 mm
- board text added: "3.3V"
- board text added: "SEM"
- board text added: "Vin"
