File: Battery with Active BMS.kicad_sch (KiCad schematic)
At the start: 83 parts, among them J1 B7B-EH-A(LF)(SN), J2 B7B-EH-A(LF)(SN), J3 B7B-EH-A(LF)(SN), P1 22-28-4033, P2 61300511121, P3 61300811121, Q1 NMOS, Q2 NMOS, U1 TLI4971, U2 ARDUINO_PRO_MINI, U3 MPC3008, U4 TC4428CPA, U5 LM78M05CT/NOPB

Commit message: V0.1 Upload
Parts:
- added P5: 22-28-4033, Connector_PinHeader_2.54mm:PinHeader_2x02_P2.54mm_Vertical, symbol Battery with Active BMS-altium-import:root_2_CN-1P-M-R3
- P3: footprint Connector_PinHeader_2.54mm:PinHeader_2x07_P2.54mm_Vertical -> Connector_PinHeader_2.54mm:PinHeader_2x09_P2.54mm_Vertical
Connections:
- net Batt+: now also B1.1, U1.8 (IP+)
- net DTR_{ISO}: now also P2.7; no longer P2.4
- net GND: now also C1.2, C2.2, C4.2, C5.2, P1.2, P2.2, P2.4, P3.16, P3.18, P3.2, P3.4, P3.6, U1.2 (GND), P5.2, P5.4; no longer C3.2, P1.3, P2.7, P2.9, P3.11, P3.13, P3.9, U5.2 (GND)
- net OCD1: now also P5.1; no longer U2.JP7_7 (D3)
- net OCD2: now also P5.3; no longer U2.JP7_8 (D2)
- net RST_{ISO}: now also P2.9; no longer P2.5
- net RX_2: now also P3.5; no longer P3.3
- net RX_{ISO}: now also P2.3; no longer P2.2
- net TX_2: now also P3.3; no longer P3.2
- net TX_{ISO}: now also P2.5; no longer P2.3
- net at U2.JP7_6 (D4): now also P3.11; no longer P3.4
- net at U2.JP7_5 (D5): now also P3.13; no longer P3.5
- net at U2.JP7_4 (D6): now also P3.15; no longer P3.6
- net at U2.JP7_3 (D7): now also P3.17; no longer P3.7
- net at U2.JP3_1 (A6): now also P1.3; no longer P1.2
- new net: P3.7, U2.JP7_8 (D2)
- new net: P3.9, U2.JP7_7 (D3)
Other:
- note added: "Isolator"
- moved on the sheet: B1, B4, B6, C1, C2, C3, C4, C5, R1, R2, U1
