File: Battery with Active BMS.kicad_sch (KiCad schematic)
At the start: 84 parts, among them J1 B7B-EH-A(LF)(SN), J2 B7B-EH-A(LF)(SN), J3 B7B-EH-A(LF)(SN), P1 22-28-4033, P2 61300511121, P3 61300811121, P5 22-28-4033, Q1 NMOS, Q2 NMOS, U1 TLI4971, U2 ARDUINO_PRO_MINI, U3 MPC3008, U4 TC4428CPA, U5 LM78M05CT/NOPB

Commit message: BMS V1.0
Parts:
- added H1, H2, H3, H4: MountingHole_Pad, MountingHole:MountingHole_5.3mm_M5_Pad_Via, symbol Mechanical:MountingHole_Pad
- added H10, H11, H12, H5, H6, H7, H8, H9: MountingHole, MountingHole:MountingHole_2.5mm_Pad, symbol Mechanical:MountingHole
- B1, B2, B3, B4, B5, B6: footprint TerminalBlock_Wuerth:Wuerth_REDCUBE-THR_WP-THRBU_74650195_THR -> lib:M5 Screw Terminal
- C3, P1, P3, P5: now not fitted
Connections:
- net GND: now also C3.2, U5.2 (GND)
- new net Copper Conn 1: H1.1, H2.1
- new net Copper Conn 2: H3.1, H4.1
Other:
- note added: "Copper Connectors"
- note added: "Mounting"
- note removed: "DNP"
- moved on the sheet: B4, BT1, BT10, BT11, BT12, BT13, BT14, BT15, BT16, BT17, BT18, BT2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

Commit message: Battery Managment System V1.0
Parts:
- removed B4: 7461383, lib:M5 Screw Terminal, symbol Battery with Active BMS-altium-import:root_0_Screw Terminal
- removed C1, C2, C3, C4, C5: Capacitor, Capacitor_SMD:C_0805_2012Metric_Pad1.18x1.45mm_HandSolder, symbol Battery with Active BMS-altium-import:root_0_Capacitor-Symbol-1
- removed P5: 22-28-4033, Connector_PinHeader_2.54mm:PinHeader_2x02_P2.54mm_Vertical, symbol Battery with Active BMS-altium-import:root_2_CN-1P-M-R3
- removed R1, R2: Res2, Resistor_SMD:R_0805_2012Metric_Pad1.20x1.40mm_HandSolder, symbol Battery with Active BMS-altium-import:root_0_Res2
- removed R26, R27: Res2, Resistor_THT:R_Axial_DIN0207_L6.3mm_D2.5mm_P10.16mm_Horizontal, symbol Battery with Active BMS-altium-import:root_1_Res2
- removed U1: TLI4971, Package_SON:Infineon_PG-TISON-8-5, symbol Battery with Active BMS-altium-import:root_0_TLI4971
- added BT19, BT20, BT21, BT22, BT23, BT24: Battery_Cell, lib:21700, symbol Device:Battery_Cell
- added J4, J8: Conn_01x05_Pin, Connector_PinSocket_2.54mm:PinSocket_1x05_P2.54mm_Vertical, symbol Connector:Conn_01x05_Pin
- added J5, J6, J7, J9: Conn_01x01_Pin, Connector_PinSocket_2.54mm:PinSocket_1x01_P2.54mm_Vertical, symbol Connector:Conn_01x01_Pin
- added R52 (x2): 4.7k, Resistor_SMD:R_0805_2012Metric_Pad1.20x1.40mm_HandSolder, symbol Device:R
Connections:
- net +3.3V: now also J4.3 (Pin_3), J8.3 (Pin_3)
- net A7: now also P1.3; no longer P1.1
- net Batt+: no longer B1.1
- net GND: now also P3.1, P3.11, P3.13, P3.15, P3.17, P3.3, P3.5, P3.7, P3.9, J4.1 (Pin_1), J4.2 (Pin_2), J8.1 (Pin_1), J8.2 (Pin_2), R52.2, R52.2; no longer P3.10, P3.12, P3.14, P3.16, P3.18, P3.2, P3.4, P3.6, P3.8
- net RST: now also P3.6; no longer P3.1
- net RX_2: now also P3.4; no longer P3.5
- net TX_2: now also P3.2; no longer P3.3
- net at BT1.1 (+), BT2.1 (+), BT3.1 (+)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: now also BT4.1 (+), BT7.2 (-), BT8.2 (-); no longer BT4.2 (-)
- net at B3.1, BT1.2 (-), BT2.2 (-)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: now also BT4.2 (-)
- net at BT10.2 (-), BT11.2 (-), BT12.2 (-)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: now also BT5.1 (+), BT6.1 (+), BT9.2 (-), J1.5, J3.5; no longer BT9.1 (+), J1.4, J3.4
- net at B2.1, J1.1, J3.1: now also BT21.1 (+), BT22.1 (+), BT23.1 (+), BT24.1 (+); no longer BT16.1 (+), BT17.1 (+), BT18.1 (+)
- net at BT13.1 (+), BT14.1 (+), BT15.1 (+)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: now also B1.1, BT16.1 (+), J1.3, J3.3, BT19.2 (-), BT20.2 (-); no longer BT16.2 (-), J1.2, J3.2
- net at BT10.1 (+), BT11.1 (+), BT12.1 (+)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: now also BT16.2 (-), BT9.1 (+), J1.4, J3.4; no longer J1.3, J3.3
- net at U2.JP7_1 (D9), U4.4 (INB): now also R52.1
- net at U2.JP7_6 (D4): now also P3.12; no longer P3.11
- net at U2.JP7_5 (D5): now also P3.14; no longer P3.13
- net at U2.JP7_4 (D6): now also P3.16; no longer P3.15
- net at U2.JP7_3 (D7): now also P3.18; no longer P3.17
- net at U2.JP7_8 (D2): now also P3.8; no longer P3.7
- net at U2.JP7_7 (D3): now also P3.10; no longer P3.9
- net at U2.JP3_1 (A6): now also P1.1; no longer P1.3
- net at U2.JP6_1 (RAW): now also J6.1 (Pin_1)
- net at U2.JP7_2 (D8), U4.2 (INA): now also R52.1
- net AOUT: no longer names the net of R12.1
- net AOUT: now also J5.1 (Pin_1)
- net VREF renamed A_{OUT}
- net A_{OUT}: now also J4.4 (Pin_4), J8.4 (Pin_4)
- new net: BT17.1 (+), BT18.1 (+), BT19.1 (+), BT20.1 (+), BT21.2 (-), BT22.2 (-), BT23.2 (-), BT24.2 (-), J1.2, J3.2
- new net ~{FAULT}: J4.5 (Pin_5), J7.1 (Pin_1), J8.5 (Pin_5), J9.1 (Pin_1)
Other:
- note removed: "Signal Filtering"
- moved on the sheet: B6, BT10, BT11, BT12, BT13, BT14, BT15, BT16, BT17, BT18, BT4, BT5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
