File: ThermistorLayout.kicad_sch (KiCad schematic)
At the start: 7 parts, among them P4 TSW-106-07-L-D

Commit message: Battery Managment System V1.0
Connections:
- net +3.3V: now also P4.1, P4.11, P4.3, P4.5, P4.7, P4.9; no longer P4.10, P4.12, P4.2, P4.4, P4.6, P4.8
- net A0: now also P4.12; no longer P4.1
- net A1: now also P4.10; no longer P4.3
- net A2: now also P4.8; no longer P4.5
- net A3: now also P4.6; no longer P4.7
- net A4: now also P4.4; no longer P4.9
- net A5: now also P4.2; no longer P4.11
Other:
- moved on the sheet: P4
Changed lines of the file:
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@@
     )
   )
-  (symbol (lib_id "Battery with Active BMS-altium-import:ThermistorLayout_0_SMTC-TSW-106-07-X-D") (at 116.84 93.98 0) (unit 1)
+  (symbol (lib_id "Battery with Active BMS-altium-import:ThermistorLayout_0_SMTC-TSW-106-07-X-D") (at 134.62 104.14 180) (unit 1)
     (in_bom yes) (on_board yes) (dnp no)
-    (property "Reference" "P4" (at 134.874 96.266 0)
+    (property "Reference" "P4" (at 116.586 101.854 0)
       (effects (font (size 1.27 1.27)) (justify left bottom))
     )
-    (property "Value" "TSW-106-07-L-D" (at 134.874 98.806 0)
+    (property "Value" "TSW-106-07-L-D" (at 116.586 99.314 0)
       (effects (font (size 1.27 1.27)) (justify left bottom))
     )
-    (property "Footprint" "Connector_PinHeader_2.54mm:PinHeader_2x06_P2.54mm_Vertical" (at 116.84 93.98 0)
+    (property "Footprint" "Connector_PinHeader_2.54mm:PinHeader_2x06_P2.54mm_Vertical" (at 134.62 104.14 0)
       (effects (font (size 1.27 1.27)) hide)
     )
-    (property "Datasheet" "" (at 116.84 93.98 0)
+    (property "Datasheet" "" (at 134.62 104.14 0)
       (effects (font (size 1.27 1.27)) hide)
     )
-    (property "COMPONENTLINK2DESCRIPTION" "Datasheet" (at 115.57 88.392 0)
+    (property "COMPONENTLINK2DESCRIPTION" "Datasheet" (at 135.89 109.728 0)
       (effects (font (size 1.27 1.27)) (justify left bottom) hide)
     )
-    (property "COMPONENTLINK1URL" "http://www.samtec.com" (at 115.57 88.392 0)
+    (property "COMPONENTLINK1URL" "http://www.samtec.com" (at 135.89 109.728 0)
       (effects (font (size 1.27 1.27)) (justify left bottom) hide)
     )
-    (property "DATASHEETVERSION" "F-214" (at 115.57 88.392 0)
+    (property "DATASHEETVERSION" "F-214" (at 135.89 109.728 0)
       (effects (font (size 1.27 1.27)) (justify left bottom) hide)
     )
-    (property "ROHS" "True" (at 115.57 88.392 0)
+    (property "ROHS" "True" (at 135.89 109.728 0)
       (effects (font (size 1.27 1.27)) (justify left bottom) hide)
     )
-    (property "COMPONENTLINK3URL" "http://www.samtec.com/documents/webfiles/cpdf/TSW-XXX-XX-XXX-X-XX-XXX-MKT.pdf" (at 115.57 88.392 0)
+    (property "COMPONENTLINK3URL" "http://www.samtec.com/documents/webfiles/cpdf/TSW-XXX-XX-XXX-X-XX-XXX-MKT.pdf" (at 135.89 109.728 0)
       (effects (font (size 1.27 1.27)) (justify left bottom) hide)
     )
-    (property "COMPONENTLINK1DESCRIPTION" "Manufacturer URL" (at 115.57 88.392 0)
+    (property "COMPONENTLINK1DESCRIPTION" "Manufacturer URL" (at 135.89 109.728 0)
       (effects (font (size 1.27 1.27)) (justify left bottom) hide)
     )
-    (property "PACKAGEVERSION" "DM, 8/1988" (at 115.57 88.392 0)
+    (property "PACKAGEVERSION" "DM, 8/1988" (at 135.89 109.728 0)
       (effects (font (size 1.27 1.27)) (justify left bottom) hide)
     )
-    (property "PITCH" "2.54 mm" (at 115.57 88.392 0)
+    (property "PITCH" "2.54 mm" (at 135.89 109.728 0)
       (effects (font (size 1.27 1.27)) (justify left bottom) hide)
     )
-    (property "MOUNTING TECHNOLOGY" "Through-hole" (at 115.57 88.392 0)
+    (property "MOUNTING TECHNOLOGY" "Through-hole" (at 135.89 109.728 0)
       (effects (font (size 1.27 1.27)) (justify left bottom) hide)
     )
-    (property "PARTNUMBER" "TSW-106-07-L-D" (at 115.57 88.392 0)
+    (property "PARTNUMBER" "TSW-106-07-L-D" (at 135.89 109.728 0)
       (effects (font (size 1.27 1.27)) (justify left bottom) hide)
     )
-    (property "TEMPERATURE RANGE" "-55 to 125 degC" (at 115.57 88.392 0)
+    (property "TEMPERATURE RANGE" "-55 to 125 degC" (at 135.89 109.728 0)
       (effects (font (size 1.27 1.27)) (justify left bottom) hide)
     )
-    (property "MANUFACTURER" "Samtec" (at 115.57 88.392 0)
+    (property "MANUFACTURER" "Samtec" (at 135.89 109.728 0)
       (effects (font (size 1.27 1.27)) (justify left bottom) hide)
     )
-    (property "COMPONENTLINK3DESCRIPTION" "Package Specification" (at 115.57 88.392 0)
+    (property "COMPONENTLINK3DESCRIPTION" "Package Specification" (at 135.89 109.728 0)
       (effects (font (size 1.27 1.27)) (justify left bottom) hide)
     )
-    (property "ORIENTATION" "Vertical" (at 115.57 88.392 0)
+    (property "ORIENTATION" "Vertical" (at 135.89 109.728 0)
       (effects (font (size 1.27 1.27)) (justify left bottom) hide)
     )
-    (property "PACKAGEDESCRIPTION" ".025[0.64] SQ. Post Terminal Strip Assembly" (at 115.57 88.392 0)
+    (property "PACKAGEDESCRIPTION" ".025[0.64] SQ. Post Terminal Strip Assembly" (at 135.89 109.728 0)
       (effects (font (size 1.27 1.27)) (justify left bottom) hide)
     )
-    (property "PACKAGEREFERENCE" "TSW-106-07-X-D" (at 115.57 88.392 0)
+    (property "PACKAGEREFERENCE" "TSW-106-07-X-D" (at 135.89 109.728 0)
       (effects (font (size 1.27 1.27)) (justify left bottom) hide)
     )
-    (property "COMPONENTLINK2URL" "http://www.samtec.com/documents/webfiles/pdf/TSW_TH.PDF" (at 115.57 88.392 0)
+    (property "COMPONENTLINK2URL" "http://www.samtec.com/documents/webfiles/pdf/TSW_TH.PDF" (at 135.89 109.728 0)
       (effects (font (size 1.27 1.27)) (justify left bottom) hide)
     )
